Commit message: Refactorizando

File: nelen_description/urdf/nelen.urdf (robot description, URDF)
Before this commit: robot nelen, 5 links, 4 joints
Links:
- removed link world
- link base_link: geometry collision mesh filename=package://nelen_description/meshes/base_corrected.dae; visual mesh filename=package://nelen_description/meshes/base_corrected.dae
- link humero: geometry collision mesh filename=package://nelen_description/meshes/humero_corrected.dae; visual mesh filename=package://nelen_description/meshes/humero_corrected.dae
- link rc: geometry collision mesh filename=package://nelen_description/meshes/rc_corrected.dae; visual mesh filename=package://nelen_description/meshes/rc_corrected.dae
- link zeta: geometry collision mesh filename=package://nelen_description/meshes/z_corrected.dae; visual mesh filename=package://nelen_description/meshes/z_corrected.dae
